Commit message: Update robot urdf camera settings and launch files

File: src/my_robot/urdf/assistance_robot.urdf.xacro (robot description, xacro)
@@ -2,4 +2,8 @@
 <robot xmlns:xacro="http://www.ros.org/wiki/xacro"
        name="humanoid_wheeled_robot">
+  <!-- ========================================================= -->
+  <!-- PROPERTIES -->
+  <!-- ========================================================= -->
+  <xacro:property name="PI" value="3.1415926535897931"/>
   <!-- ========================================================= -->
   <!-- MATERIALS -->
@@ -34,5 +38,5 @@
   <link name="base_link">
     <visual>
-      <origin xyz="0 0 0.18"/>
+      <origin xyz="0 0 0.18" rpy="0 0 0"/>
       <geometry>
         <box size="0.65 0.55 0.36"/>
@@ -41,5 +45,5 @@
     </visual>
     <collision>
-      <origin xyz="0 0 0.18"/>
+      <origin xyz="0 0 0.18" rpy="0 0 0"/>
       <geometry>
         <box size="0.65 0.55 0.36"/>
@@ -49,11 +53,5 @@
       <origin xyz="0 0 0.18"/>
       <mass value="20.0"/>
-      <inertia
-        ixx="1.0"
-        ixy="0.0"
-        ixz="0.0"
-        iyy="1.0"
-        iyz="0.0"
-        izz="1.0"/>
+      <inertia ixx="1.0" ixy="0.0" ixz="0.0" iyy="1.0" iyz="0.0" izz="1.0"/>
     </inertial>
   </link>
@@ -78,11 +76,5 @@
       <origin xyz="0 0 0"/>
       <mass value="2.0"/>
-      <inertia
-        ixx="0.02"
-        ixy="0.0"
-        ixz="0.0"
-        iyy="0.02"
-        iyz="0.0"
-        izz="0.02"/>
+      <inertia ixx="0.02" ixy="0.0" ixz="0.0" iyy="0.02" iyz="0.0" izz="0.02"/>
     </inertial>
   </link>
@@ -113,11 +105,5 @@
       <origin xyz="0 0 0"/>
       <mass value="2.0"/>
-      <inertia
-        ixx="0.02"
-        ixy="0.0"
-        ixz="0.0"
-        iyy="0.02"
-        iyz="0.0"
-        izz="0.02"/>
+      <inertia ixx="0.02" ixy="0.0" ixz="0.0" iyy="0.02" iyz="0.0" izz="0.02"/>
     </inertial>
   </link>
@@ -146,11 +132,5 @@
       <origin xyz="0 0 0"/>
       <mass value="0.5"/>
-      <inertia
-        ixx="0.001"
-        ixy="0.0"
-        ixz="0.0"
-        iyy="0.001"
-        iyz="0.0"
-        izz="0.001"/>
+      <inertia ixx="0.001" ixy="0.0" ixz="0.0" iyy="0.001" iyz="0.0" izz="0.001"/>
     </inertial>
   </link>
@@ -178,11 +158,5 @@
       <origin xyz="0 0 0"/>
       <mass value="0.5"/>
-      <inertia
-        ixx="0.001"
-        ixy="0.0"
-        ixz="0.0"
-        iyy="0.001"
-        iyz="0.0"
-        izz="0.001"/>
+      <inertia ixx="0.001" ixy="0.0" ixz="0.0" iyy="0.001" iyz="0.0" izz="0.001"/>
     </inertial>
   </link>
@@ -197,5 +171,5 @@
   <link name="torso_link">
     <visual>
-      <origin xyz="0 0 0.42"/>
+      <origin xyz="0 0 0.42" rpy="0 0 0"/>
       <geometry>
         <box size="0.48 0.50 0.84"/>
@@ -204,5 +178,5 @@
     </visual>
     <collision>
-      <origin xyz="0 0 0.42"/>
+      <origin xyz="0 0 0.42" rpy="0 0 0"/>
       <geometry>
         <box size="0.48 0.50 0.84"/>
@@ -212,11 +186,5 @@
       <origin xyz="0 0 0.42"/>
       <mass value="12.0"/>
-      <inertia
-        ixx="0.8"
-        ixy="0.0"
-        ixz="0.0"
-        iyy="0.8"
-        iyz="0.0"
-        izz="0.6"/>
+      <inertia ixx="0.8" ixy="0.0" ixz="0.0" iyy="0.8" iyz="0.0" izz="0.6"/>
     </inertial>
   </link>
@@ -224,12 +192,12 @@
     <parent link="base_link"/>
     <child link="torso_link"/>
-    <origin xyz="0 0 0.36"/>
-  </joint>
-  <!-- ========================================================= -->
-  <!-- HEAD -->
+    <origin xyz="0 0 0.36" rpy="0 0 0"/>
+  </joint>
+  <!-- ========================================================= -->
+  <!-- HEAD (Shifted Forward to Front Face) -->
   <!-- ========================================================= -->
   <link name="head_link">
     <visual>
-      <origin xyz="0 0 0.14"/>
+      <origin xyz="0 0 0" rpy="0 0 0"/>
       <geometry>
         <box size="0.28 0.32 0.28"/>
@@ -238,5 +206,5 @@
     </visual>
     <collision>
-      <origin xyz="0 0 0.14"/>
+      <origin xyz="0 0 0" rpy="0 0 0"/>
       <geometry>
         <box size="0.28 0.32 0.28"/>
@@ -244,44 +212,53 @@
     </collision>
     <inertial>
-      <origin xyz="0 0 0.14"/>
+      <origin xyz="0 0 0"/>
       <mass value="2.0"/>
-      <inertia
-        ixx="0.08"
-        ixy="0.0"
-        ixz="0.0"
-        iyy="0.08"
-        iyz="0.0"
-        izz="0.08"/>
-    </inertial>
-  </link>
-  <!-- ========================================================= -->
-  <!-- NECK -->
-  <!-- ========================================================= -->
+      <inertia ixx="0.08" ixy="0.0" ixz="0.0" iyy="0.08" iyz="0.0" izz="0.08"/>
+    </inertial>
+  </link>
   <joint name="neck_joint" type="revolute">
     <parent link="torso_link"/>
     <child link="head_link"/>
-    <origin xyz="0 0 0.84"/>
+    <!-- تم تقديم الرأس للأمام قليلاً ليكون في وجه الروبوت -->
+    <origin xyz="0.10 0 0.84" rpy="0 0 0"/>
     <axis xyz="0 0 1"/>
-    <limit
-      lower="-1.57"
-      upper="1.57"
-      effort="10"
-      velocity="1.0"/>
-  </joint>
-  <!-- ========================================================= -->
-  <!-- 6 DOF ARM -->
-  <!-- ========================================================= -->
-  <!--
-    ZERO POSE:
-    q1 = 0
-    q2 = 0
-    q3 = 0
-    q4 = 0
-    q5 = 0
-    q6 = 0
-    Upper arm + forearm + wrist point along +X.
-  -->
-  <!-- ========================================================= -->
-  <!-- 1. SHOULDER PITCH -->
+    <limit lower="0.0" upper="0.0" effort="10" velocity="1.0"/>
+  </joint>
+  <!-- ========================================================= -->
+  <!-- RGB-D CAMERA -->
+  <!-- ========================================================= -->
+  <link name="camera_link">
+    <visual>
+      <origin xyz="0 0 0" rpy="0 0 0"/>
+      <geometry>
+        <box size="0.06 0.12 0.05"/>
+      </geometry>
+      <material name="black"/>
+    </visual>
+    <collision>
+      <origin xyz="0 0 0" rpy="0 0 0"/>
+      <geometry>
+        <box size="0.06 0.12 0.05"/>
+      </geometry>
+    </collision>
+    <inertial>
+      <origin xyz="0 0 0"/>
+      <mass value="0.15"/>
+      <inertia ixx="0.001" ixy="0.0" ixz="0.0" iyy="0.001" iyz="0.0" izz="0.001"/>
+    </inertial>
+  </link>
+  <link name="camera_optical_frame"/>
+  <joint name="camera_joint" type="fixed">
+    <parent link="head_link"/>
+    <child link="camera_link"/>
+    <origin xyz="0.15 0 0" rpy="0 0 0"/>
+  </joint>
+  <joint name="camera_optical_joint" type="fixed">
+    <parent link="camera_link"/>
+    <child link="camera_optical_frame"/>
+    <origin xyz="0 0 0" rpy="-1.5708 0 -1.5708"/>
+  </joint>
+  <!-- ========================================================= -->
+  <!-- 6 DOF ARM (Corrected Front Shoulder Mount) -->
   <!-- ========================================================= -->
   <link name="shoulder_pitch_link">
@@ -289,5 +266,5 @@
       <origin xyz="0 0 0" rpy="0 1.5708 0"/>
       <geometry>
-        <cylinder radius="0.085" length="0.14"/>
+        <cylinder radius="0.06" length="0.10"/>
       </geometry>
       <material name="orange"/>
@@ -296,5 +273,5 @@
       <origin xyz="0 0 0" rpy="0 1.5708 0"/>
       <geometry>
-        <cylinder radius="0.085" length="0.14"/>
+        <cylinder radius="0.06" length="0.10"/>
       </geometry>
     </collision>
@@ -302,11 +279,5 @@
       <origin xyz="0 0 0"/>
       <mass value="0.8"/>
-      <inertia
-        ixx="0.012"
-        ixy="0.0"
-        ixz="0.0"
-        iyy="0.012"
-        iyz="0.0"
-        izz="0.012"/>
+      <inertia ixx="0.012" ixy="0.0" ixz="0.0" iyy="0.012" iyz="0.0" izz="0.012"/>
     </inertial>
   </link>
@@ -314,27 +285,24 @@
     <parent link="torso_link"/>
     <child link="shoulder_pitch_link"/>
-    <origin xyz="0 0.32 0.68" rpy="0 0 0"/>
+    <!-- تم ضبط مكان الكتف ليخرج من مقدمة وجانب التورسو بوضوح -->
+    <origin xyz="0.12 0.28 0.60" rpy="0 0 0"/>
     <axis xyz="0 1 0"/>
-    <limit
-      lower="-1.57"
-      upper="1.57"
-      effort="40"
-      velocity="1.5"/>
-  </joint>
-  <!-- ========================================================= -->
-  <!-- 2. SHOULDER ROLL -->
+    <limit lower="-1.57" upper="1.57" effort="40" velocity="1.5"/>
+  </joint>
+  <!-- ========================================================= -->
+  <!-- SHOULDER ROLL -->
   <!-- ========================================================= -->
   <link name="shoulder_roll_link">
     <visual>
-      <origin xyz="0 0 0"/>
-      <geometry>
-        <cylinder radius="0.075" length="0.14"/>
+      <origin xyz="0 0 0" rpy="0 0 0"/>
+      <geometry>
+        <cylinder radius="0.055" length="0.10"/>
       </geometry>
       <material name="blue"/>
     </visual>
     <collision>
-      <origin xyz="0 0 0"/>
-      <geometry>
-        <cylinder radius="0.075" length="0.14"/>
+      <origin xyz="0 0 0" rpy="0 0 0"/>
+      <geometry>
+        <cylinder radius="0.055" length="0.10"/>
       </geometry>
     </collision>
@@ -342,11 +310,5 @@
       <origin xyz="0 0 0"/>
       <mass value="1.0"/>
-      <inertia
-        ixx="0.015"
-        ixy="0.0"
-        ixz="0.0"
-        iyy="0.015"
-        iyz="0.0"
-        izz="0.015"/>
+      <inertia ixx="0.015" ixy="0.0" ixz="0.0" iyy="0.015" iyz="0.0" izz="0.015"/>
     </inertial>
   </link>
@@ -356,37 +318,27 @@
     <origin xyz="0 0 0" rpy="0 0 0"/>
     <axis xyz="1 0 0"/>
-    <limit
-      lower="-1.57"
-      upper="1.57"
-      effort="40"
-      velocity="1.5"/>
-  </joint>
-  <!-- ========================================================= -->
-  <!-- 3. SHOULDER YAW / UPPER ARM -->
+    <limit lower="-1.57" upper="1.57" effort="40" velocity="1.5"/>
+  </joint>
+  <!-- ========================================================= -->
+  <!-- UPPER ARM -->
   <!-- ========================================================= -->
   <link name="upper_arm_link">
     <visual>
-      <origin xyz="0.22 0 0" rpy="0 1.5708 0"/>
-      <geometry>
-        <cylinder radius="0.065" length="0.44"/>
+      <origin xyz="0.15 0 0" rpy="0 1.5708 0"/>
+      <geometry>
+        <cylinder radius="0.045" length="0.30"/>
       </geometry>
       <material name="white"/>
     </visual>
     <collision>
-      <origin xyz="0.22 0 0" rpy="0 1.5708 0"/>
-      <geometry>
-        <cylinder radius="0.065" length="0.44"/>
-      </geometry>
-    </collision>
-    <inertial>
-      <origin xyz="0.22 0 0"/>
+      <origin xyz="0.15 0 0" rpy="0 1.5708 0"/>
+      <geometry>
+        <cylinder radius="0.045" length="0.30"/>
+      </geometry>
+    </collision>
+    <inertial>
+      <origin xyz="0.15 0 0"/>
       <mass value="1.8"/>
-      <inertia
-        ixx="0.03"
-        ixy="0.0"
-        ixz="0.0"
-        iyy="0.03"
-        iyz="0.0"
-        izz="0.03"/>
+      <inertia ixx="0.03" ixy="0.0" ixz="0.0" iyy="0.03" iyz="0.0" izz="0.03"/>
     </inertial>
   </link>
@@ -396,37 +348,27 @@
     <origin xyz="0 0 0" rpy="0 0 0"/>
     <axis xyz="0 0 1"/>
-    <limit
-      lower="-3.14159"
-      upper="3.14159"
-      effort="30"
-      velocity="1.5"/>
-  </joint>
-  <!-- ========================================================= -->
-  <!-- 4. ELBOW PITCH -->
+    <limit lower="-3.14159" upper="3.14159" effort="30" velocity="1.5"/>
+  </joint>
+  <!-- ========================================================= -->
+  <!-- FOREARM / ELBOW -->
   <!-- ========================================================= -->
   <link name="forearm_link">
     <visual>
-      <origin xyz="0.20 0 0" rpy="0 1.5708 0"/>
-      <geometry>
-        <cylinder radius="0.05" length="0.40"/>
+      <origin xyz="0.15 0 0" rpy="0 1.5708 0"/>
+      <geometry>
+        <cylinder radius="0.04" length="0.30"/>
       </geometry>
       <material name="orange"/>
     </visual>
     <collision>
-      <origin xyz="0.20 0 0" rpy="0 1.5708 0"/>
-      <geometry>
-        <cylinder radius="0.05" length="0.40"/>
-      </geometry>
-    </collision>
-    <inertial>
-      <origin xyz="0.20 0 0"/>
+      <origin xyz="0.15 0 0" rpy="0 1.5708 0"/>
+      <geometry>
+        <cylinder radius="0.04" length="0.30"/>
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